Commit message: Removed rotation from depth camera frame

File: clearpath_sensors_description/urdf/intel_realsense.urdf.xacro (robot description, xacro)
@@ -82,5 +82,5 @@
         <link name="${name}_depth_frame"/>
         <joint name="${name}_depth_optical_joint" type="fixed">
-          <origin xyz="0 0 0" rpy="${-M_PI/2} 0 ${-M_PI/2}" />
+          <origin xyz="0 0 0" rpy="0 0 0" />
           <parent link="${name}_depth_frame" />
           <child link="${name}_depth_optical_frame" />
@@ -108,5 +108,5 @@
         <link name="${name}_infra2_frame"/>
         <joint name="${name}_infra2_optical_joint" type="fixed">
-          <origin xyz="0 0 0" rpy="${-M_PI/2} 0 ${-M_PI/2}" />
+          <origin xyz="0 0 0" rpy="0 0 0" />
           <parent link="${name}_infra2_frame" />
           <child link="${name}_infra2_optical_frame" />
@@ -121,5 +121,5 @@
         <link name="${name}_color_frame"/>
         <joint name="${name}_color_optical_joint" type="fixed">
-          <origin xyz="0 0 0" rpy="${-M_PI/2} 0 ${-M_PI/2}" />
+          <origin xyz="0 0 0" rpy="0 0 0" />
           <parent link="${name}_color_frame" />
           <child link="${name}_color_optical_frame" />
